Commit message: nuevo URDF

File: taurus_description/urdf/taurus.urdf (robot description, URDF)
Before this commit: robot taurus, 7 links, 6 joints
Links:
- removed link base_footprint
- removed link caster_ball_link
- removed link imu_link
- removed link scan_link
- removed link wheel_left_link
- removed link wheel_right_link
- added link Base_castor_link, mass 0.00033463; collision mesh filename=package://taurus_description/meshes/Base_castor_link.STL; visual mesh filename=package://taurus_description/meshes/Base_castor_link.STL
- added link Caster_ball_link, mass 0.002; collision mesh filename=package://taurus_description/meshes/Caster_ball_link.STL; visual mesh filename=package://taurus_description/meshes/Caster_ball_link.STL
- added link Rueda_derecha_link, mass 0.03; collision mesh filename=package://taurus_description/meshes/Rueda_derecha_link.STL; visual mesh filename=package://taurus_description/meshes/Rueda_derecha_link.STL
- added link Rueda_izquierda_link, mass 0.03; collision mesh filename=package://taurus_description/meshes/Rueda_izquierda_link.STL; visual mesh filename=package://taurus_description/meshes/Rueda_izquierda_link.STL
- added link Scan_link, mass 0.0055715; collision mesh filename=package://taurus_description/meshes/Scan_link.STL; visual mesh filename=package://taurus_description/meshes/Scan_link.STL
- added link base_link_ground
- link base_link: mass 0.3 -> 0.109923704165007
Joints:
- removed joint base_joint
- removed joint caster_ball_joint
- removed joint imu_joint
- removed joint scan_joint
- removed joint wheel_left_joint
- removed joint wheel_right_joint
- added joint Base_castor_joint: type fixed, parent base_link, child Base_castor_link, origin xyz=0.056575 0 0.0034302 rpy=0 0 0, axis 0 0 0
- added joint Caster_ball_joint: type continuous, parent Base_castor_link, child Caster_ball_link, origin xyz=-1.325E-05 -3.8318E-05 -0.004121 rpy=-1.5708 0 0, axis 1 0 1
- added joint Rueda_derecha_joint: type continuous, parent base_link, child Rueda_derecha_link, origin xyz=-0.0043003 -0.059687 0.0079472 rpy=-1.5708 0 0, axis 0 0 1
- added joint Rueda_izquierda_joint: type continuous, parent base_link, child Rueda_izquierda_link, origin xyz=-0.0043291 0.036579 0.0080704 rpy=-1.5708 0 0, axis 0 0 1
- added joint Scan_joint: type fixed, parent base_link, child Scan_link, origin xyz=0.03982 9.4804E-05 0.016343 rpy=0 0 0, axis 0 0 0
- added joint ground_base_joint: type fixed, parent base_link_ground, child base_link, origin xyz=0.0 0.0 0.0 rpy=0.0 0.0 0.0

File: taurus_description/urdf/taurus.urdf.xacro (robot description, xacro)
@@ -5,14 +5,4 @@
     <!-- Include ros2_control Plugins -->
     <xacro:include filename="$(find taurus_description)/urdf/taurus_ros2_control.xacro" />
-    <!-- Colors -->
-    <material name="black">
-        <color rgba="0.4 0.4 0.4 1.0"/>
-    </material>
-    <material name="white">
-        <color rgba="1.0 1.0 1.0 1.0"/>
-    </material>
-    <material name="orange">
-        <color rgba="${255/255} ${190/255} ${50/255} 0.98"/>
-    </material>
 <!--link name="odom_frame"/>
     <joint name="odom_joint" type="fixed">
@@ -21,191 +11,321 @@
       <origin xyz="0.0 0.0 0.0" rpy="0.0 0.0 0.0" />
     </joint-->
-    <!-- Links -->
-    <link name="base_footprint"/>
-    <link name="base_link">
-        <inertial>
-            <origin xyz="0.003868358578296 -0.000158188357109068 0.0163891387106582" rpy="0 0 0" />
-            <mass value="0.3" />
-            <inertia
-            ixx="0.0001"
-            ixy="0"
-            ixz="0"
-            iyy="0.0003"
-            iyz="0"
-            izz="0.0002" />
-        </inertial>
-        <visual>
-            <origin xyz="0 0 0" rpy="0 0 0" />
-            <geometry>
-            <mesh filename="package://taurus_description/meshes/base_link.STL" />
-            </geometry>
-            <material name="orange"/>
-        </visual>
-        <collision>
-            <origin xyz="0 0 0" rpy="0 0 0" />
-            <geometry>
-                <mesh filename="package://taurus_description/meshes/base_link.STL" />
-            </geometry>
-        </collision>
-    </link>
-    <joint name="base_joint" type="fixed">
-        <parent link="base_footprint"/>
-        <child link="base_link"/>
-        <origin xyz="0.0 0.0 0.000" rpy="0 0 0"/>
-    </joint>
-    <link name="wheel_left_link">
-        <inertial>
-            <origin xyz="-2.0625E-05 -6.8524E-05 0.010935"
-             rpy="0 0 0" />
-            <mass value="0.3" />
-            <inertia
-            ixx="0.00002"
-            ixy="0"
-            ixz="0"
-            iyy="0.00002"
-            iyz="0"
-            izz="0.0001" />
-        </inertial>
-        <visual>
-            <origin xyz="0 0 0" rpy="0 0 0" />
-            <geometry>
-                <mesh filename="package://taurus_description/meshes/wheel_left_tire.STL" />
-            </geometry>
-            <material name="black" />
-        </visual>
-        <collision>
-            <origin xyz="0 0 0" rpy="0 0 0" />
-            <geometry>
-                <cylinder length="0.018" radius="0.016"/>
-            </geometry>
-        </collision>
-    </link>
-    <joint name="wheel_left_joint" type="continuous">
-        <origin
-        xyz="-0.0033479 0.03711 0.0080001"
-        rpy="-1.5708 0 -0.0018302" />
-        <parent link="base_link" />
-        <child link="wheel_left_link" />
-        <axis xyz="0 0 1" />
-    </joint>
-    <link name="wheel_right_link">
-        <inertial>
-            <origin
-              xyz="2.1073E-05 6.8519E-05 -0.010935"
-              rpy="0 0 0" />
-            <mass value="0.3" />
-            <inertia
-            ixx="0.00002"
-            ixy="0"
-            ixz="0"
-            iyy="0.00002"
-            iyz="0"
-            izz="0.0001" />
-        </inertial>
-        <visual>
-            <origin xyz="0 0 0" rpy="0 0 0" />
-            <geometry>
-                <mesh filename="package://taurus_description/meshes/wheel_right_tire.STL" />
-            </geometry>
-            <material name="black" />
-        </visual>
-        <collision>
-            <origin xyz="0 0 0" rpy="0 0 0" />
-            <geometry>
-                <cylinder length="0.018" radius="0.016"/>
-            </geometry>
-        </collision>
-    </link>
-    <joint name="wheel_right_joint" type="continuous">
-        <origin
-          xyz="-0.0033372 -0.037239 0.0080194"
-          rpy="-1.5708 0 -0.0018302" />
-        <parent link="base_link" />
-        <child link="wheel_right_link" />
-        <axis xyz="0 0 1" />
-    </joint>
-    <link name="caster_ball_link">
-        <inertial>
-            <origin
-             xyz="0 1.3878E-17 0"
-             rpy="0 0 0" />
-            <mass value="0.2" />
-            <inertia
-            ixx="0.0004"
-            ixy="0"
-            ixz="0"
-            iyy="0.0004"
-            iyz="0"
-            izz="0.00001" />
-        </inertial>
-        <visual>
-            <origin xyz="0 0 0" rpy="0 0 0" />
-            <geometry>
-                <mesh filename="package://taurus_description/meshes/caster_ball.STL" />
-            </geometry>
-            <material name="white"/>
-        </visual>
-        <collision>
-            <origin xyz="0 0 0" rpy="0 0 0" />
-            <geometry>
-                <mesh filename="package://taurus_description/meshes/caster_ball.STL" />
-            </geometry>
-        </collision>
-    </link>
-    <joint name="caster_ball_joint" type="fixed">
-        <origin
-         xyz="0.057569 -4.6108E-05 -0.00046991"
-         rpy="-1.5708 0 -0.0018302" />
-        <parent link="base_link" />
-        <child link="caster_ball_link" />
-    </joint>
-    <link name="scan_link">
-        <inertial>
-            <origin
-             xyz="0 0 0"
-             rpy="0 0 0" />
-            <mass value="0.1" />
-            <inertia
-            ixx="0.00001"
-            ixy="0"
-            ixz="0"
-            iyy="0.000001"
-            iyz="0"
-            izz="0.000001" />
-        </inertial>
-        <visual>
-            <origin xyz="0 0 0" rpy="0 0 0" />
-            <geometry>
-                <mesh filename="package://taurus_description/meshes/scan_link.STL" />
-            </geometry>
-            <material name="black"/>
-        </visual>
-        <collision>
-            <origin xyz="0 0 0" rpy="0 0 0" />
-            <geometry>
-                <mesh filename="package://taurus_description/meshes/scan_link.STL" />
-            </geometry>
-        </collision>
-    </link>
-    <joint name="scan_joint" type="fixed">
-        <origin
-        xyz="0.040761 0.00011153 0.016498"
-        rpy="0 0 -0.0018302" />
-        <parent link="base_link" />
-        <child link="scan_link" />
-        <axis xyz="0 0 1" />
-    </joint>
-    <joint name="imu_joint" type="fixed">
-        <parent link="base_link"/>
-        <child link="imu_link"/>
-        <origin xyz="0 0 0" rpy="0 0 0"/>
-    </joint>
-    <link name="imu_link"/>
+  <link
+    name="base_link">
+    <inertial>
+      <origin
+        xyz="0.00293768617847148 -0.000180932444542536 0.0163820289331232"
+        rpy="0 0 0" />
+      <mass
+        value="0.109923704165007" />
+      <inertia
+        ixx="0.0001"
+        ixy="0"
+        ixz="0"
+        iyy="0.0003"
+        iyz="0"
+        izz="0.0002" />
+    </inertial>
+    <visual>
+      <origin
+        xyz="0 0 0"
+        rpy="0 0 0" />
+      <geometry>
+        <mesh
+          filename="package://taurus_description/meshes/base_link.STL" />
+      </geometry>
+      <material
+        name="">
+        <color
+          rgba="0.745098039215686 0.737254901960784 0.729411764705882 1" />
+      </material>
+    </visual>
+    <collision>
+      <origin
+        xyz="0 0 0"
+        rpy="0 0 0" />
+      <geometry>
+        <mesh
+          filename="package://taurus_description/meshes/base_link.STL" />
+      </geometry>
+    </collision>
+  </link>
+  <link name="base_link_ground"/>
+  <joint name="ground_base_joint" type="fixed">
+    <parent link="base_link_ground" />
+    <child link = "base_link" />
+    <origin xyz="0.0 0.0 0.0" rpy="0.0 0.0 0.0" />
+  </joint>
+  <link
+    name="Rueda_derecha_link">
+    <inertial>
+      <origin
+        xyz="-2.2882E-06 5.0601E-05 0.012107"
+        rpy="0 0 0" />
+      <mass
+        value="0.03" />
+      <inertia
+        ixx="0.00002"
+        ixy="0"
+        ixz="0"
+        iyy="0.00002"
+        iyz="0"
+        izz="0.0001" />
+    </inertial>
+    <visual>
+      <origin
+        xyz="0 0 0"
+        rpy="0 0 0" />
+      <geometry>
+        <mesh
+          filename="package://taurus_description/meshes/Rueda_derecha_link.STL" />
+      </geometry>
+      <material
+        name="">
+        <color
+          rgba="0.29804 0.29804 0.29804 1" />
+      </material>
+    </visual>
+    <collision>
+      <origin
+        xyz="0 0 0"
+        rpy="0 0 0" />
+      <geometry>
+        <mesh
+          filename="package://taurus_description/meshes/Rueda_derecha_link.STL" />
+      </geometry>
+    </collision>
+  </link>
+  <joint
+    name="Rueda_derecha_joint"
+    type="continuous">
+    <origin
+      xyz="-0.0043003 -0.059687 0.0079472"
+      rpy="-1.5708 0 0" />
+    <parent
+      link="base_link" />
+    <child
+      link="Rueda_derecha_link" />
+    <axis
+      xyz="0 0 1" />
+  </joint>
+  <link
+    name="Rueda_izquierda_link">
+    <inertial>
+      <origin
+        xyz="-2.0761E-06 -8.4779E-05 0.010976"
+        rpy="0 0 0" />
+      <mass
+        value="0.03" />
+      <inertia
+        ixx="0.00002"
+        ixy="0"
+        ixz="0"
+        iyy="0.00002"
+        iyz="0"
+        izz="0.0001" />
+    </inertial>
+    <visual>
+      <origin
+        xyz="0 0 0"
+        rpy="0 0 0" />
+      <geometry>
+        <mesh
+          filename="package://taurus_description/meshes/Rueda_izquierda_link.STL" />
+      </geometry>
+      <material
+        name="">
+        <color
+          rgba="0.29804 0.29804 0.29804 1" />
+      </material>
+    </visual>
+    <collision>
+      <origin
+        xyz="0 0 0"
+        rpy="0 0 0" />
+      <geometry>
+        <mesh
+          filename="package://taurus_description/meshes/Rueda_izquierda_link.STL" />
+      </geometry>
+    </collision>
+  </link>
+  <joint
+    name="Rueda_izquierda_joint"
+    type="continuous">
+    <origin
+      xyz="-0.0043291 0.036579 0.0080704"
+      rpy="-1.5708 0 0" />
+    <parent
+      link="base_link" />
+    <child
+      link="Rueda_izquierda_link" />
+    <axis
+      xyz="0 0 1" />
+  </joint>
+  <link
+    name="Scan_link">
+    <inertial>
+      <origin
+        xyz="0.010059 -0.00088382 0.000124"
+        rpy="0 0 0" />
+      <mass
+        value="0.0055715" />
+      <inertia
+        ixx="5.6499E-07"
+        ixy="3.6334E-08"
+        ixz="3.4462E-09"
+        iyy="2.3592E-07"
+        iyz="-1.4863E-09"
+        izz="6.4738E-07" />
+    </inertial>
+    <visual>
+      <origin
+        xyz="0 0 0"
+        rpy="0 0 0" />
+      <geometry>
+        <mesh
+          filename="package://taurus_description/meshes/Scan_link.STL" />
+      </geometry>
+      <material
+        name="">
+        <color
+          rgba="0.79216 0.81961 0.93333 1" />
+      </material>
+    </visual>
+    <collision>
+      <origin
+        xyz="0 0 0"
+        rpy="0 0 0" />
+      <geometry>
+        <mesh
+          filename="package://taurus_description/meshes/Scan_link.STL" />
+      </geometry>
+    </collision>
+  </link>
+  <joint
+    name="Scan_joint"
+    type="fixed">
+    <origin
+      xyz="0.03982 9.4804E-05 0.016343"
+      rpy="0 0 0" />
+    <parent
+      link="base_link" />
+    <child
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