Commit message: nodo de mapeo cartographer

File: src/taurus_description/urdf/taurus.urdf (robot description, URDF)
Before this commit: robot taurus, 8 links, 7 joints
Links:
- removed link Base_castor_link
- removed link Caster_ball_link
- removed link Rueda_derecha_link
- removed link Rueda_izquierda_link
- removed link Scan_link
- removed link base_link_ground
- added link base_castor_link, mass 0.00033463; collision mesh filename=package://taurus_description/meshes/base_castor_link.STL; visual mesh filename=package://taurus_description/meshes/base_castor_link.STL
- added link base_footprint
- added link caster_ball_link, mass 0.06; collision sphere radius=0.005; visual mesh filename=package://taurus_description/meshes/caster_ball_link.STL
- added link rueda_derecha_link, mass 0.08; collision cylinder length=0.016 radius=0.015; visual mesh filename=package://taurus_description/meshes/rueda_derecha_link.STL
- added link rueda_izquierda_link, mass 0.08; collision cylinder length=0.016 radius=0.015; visual mesh filename=package://taurus_description/meshes/rueda_izquierda_link.STL
- added link scan_link, mass 0.0055715; collision mesh filename=package://taurus_description/meshes/scan_link.STL; visual mesh filename=package://taurus_description/meshes/scan_link.STL
Joints:
- removed joint Base_castor_joint
- removed joint Caster_ball_joint
- removed joint Rueda_derecha_joint
- removed joint Rueda_izquierda_joint
- removed joint Scan_joint
- removed joint ground_base_joint
- added joint base_castor_joint: type fixed, parent base_link, child base_castor_link, origin xyz=0.056575 0 0.0034302 rpy=0 0 0, axis 0 0 0
- added joint caster_ball_joint: type fixed, parent base_castor_link, child caster_ball_link, origin xyz=-1.325E-05 -3.8318E-05 -0.004121 rpy=-1.5708 0 0, axis 0 0 0, limit lower=0 upper=0 effort=0 velocity=0
- added joint ground_joint: type fixed, parent base_footprint, child base_link, origin xyz=0 0 0.005 rpy=0 0 0
- added joint rueda_derecha_joint: type continuous, parent base_link, child rueda_derecha_link, origin xyz=-0.0043003 -0.059687 0.0079472 rpy=-1.5708 0 0, axis 0 0 1
- added joint rueda_izquierda_joint: type continuous, parent base_link, child rueda_izquierda_link, origin xyz=-0.0043291 0.036579 0.0080704 rpy=-1.5708 0 0, axis 0 0 1
- added joint scan_joint: type fixed, parent base_link, child scan_link, origin xyz=0.03982 9.4804E-05 0.016343 rpy=0 -0.0208 0, axis 0 0 0
- joint imu_joint: axis 1 0 0 -> (none)

File: src/taurus_description/urdf/taurus.urdf.xacro (robot description, xacro)
@@ -1,10 +1,10 @@
 <?xml version="1.0"?>
 <robot name="taurus" xmlns:xacro="http://ros.org/wiki/xacro">
-<!--link name="odom_frame"/>
-    <joint name="odom_joint" type="fixed">
-      <parent link="odom_frame" />
-      <child link = "base_link" />
-      <origin xyz="0.0 0.0 0.0" rpy="0.0 0.0 0.0" />
-    </joint-->
+  <!--link name="odom_frame"/>
+  <joint name="odom_joint" type="fixed">
+    <parent link="odom_frame" />
+    <child link = "base_link" />
+    <origin xyz="0.0 0.0 0.0" rpy="0.0 0.0 0.0" />
+  </joint-->
   <link
     name="base_link">
@@ -47,9 +47,9 @@
     </collision>
   </link>
-  <link name="base_link_ground"/>
-  <joint name="ground_base_joint" type="fixed">
-    <parent link="base_link_ground" />
+  <link name="base_footprint"/>
+  <joint name="ground_joint" type="fixed">
+    <parent link="base_footprint" />
     <child link = "base_link" />
-    <origin xyz="0.0 0.0 0.0" rpy="0.0 0.0 0.0" />
+    <origin xyz="0 0 0.005" rpy="0 0 0"/>
   </joint>
   <gazebo reference="base_link">
@@ -58,8 +58,7 @@
     <kp>1000000</kp>
     <kd>1</kd>
-    <material>Gazebo/Yellow</material>
-  </gazebo>
-  <link
-    name="Rueda_derecha_link">
+  </gazebo>
+  <link
+    name="rueda_derecha_link">
     <inertial>
       <origin
@@ -67,20 +66,20 @@
         rpy="0 0 0" />
       <mass
-        value="0.03" />
-      <inertia
-        ixx="0.00002"
+        value="0.08" />
+      <inertia
+        ixx="0.000002"
         ixy="0"
         ixz="0"
-        iyy="0.00002"
+        iyy="0.000002"
         iyz="0"
-        izz="0.0001" />
-    </inertial>
-    <visual>
-      <origin
-        xyz="0 0 0"
-        rpy="0 0 0" />
-      <geometry>
-        <mesh
-          filename="package://taurus_description/meshes/Rueda_derecha_link.STL" />
+        izz="0.00001" />
+    </inertial>
+    <visual>
+      <origin
+        xyz="0 0 0"
+        rpy="0 0 0" />
+      <geometry>
+        <mesh
+          filename="package://taurus_description/meshes/rueda_derecha_link.STL" />
       </geometry>
       <material
@@ -95,11 +94,10 @@
         rpy="0 0 0" />
       <geometry>
-        <mesh
-          filename="package://taurus_description/meshes/Rueda_derecha_link.STL" />
-      </geometry>
-    </collision>
-  </link>
-  <joint
-    name="Rueda_derecha_joint"
+        <cylinder radius="0.015" length="0.016"/>
+      </geometry>
+    </collision>
+  </link>
+  <joint
+    name="rueda_derecha_joint"
     type="continuous">
     <origin
@@ -109,17 +107,16 @@
       link="base_link" />
     <child
-      link="Rueda_derecha_link" />
+      link="rueda_derecha_link" />
     <axis
       xyz="0 0 1" />
   </joint>
-    <gazebo reference="Rueda_derecha_link">
+    <gazebo reference="rueda_derecha_link">
     <mu1>200</mu1>
     <mu2>200</mu2>
     <kp>1000000</kp>
     <kd>1</kd>
-    <material>Gazebo/Gray</material>
-  </gazebo>
-  <link
-    name="Rueda_izquierda_link">
+  </gazebo>
+  <link
+    name="rueda_izquierda_link">
     <inertial>
       <origin
@@ -127,20 +124,20 @@
         rpy="0 0 0" />
       <mass
-        value="0.03" />
-      <inertia
-        ixx="0.00002"
+        value="0.08" />
+      <inertia
+        ixx="0.000002"
         ixy="0"
         ixz="0"
-        iyy="0.00002"
+        iyy="0.000002"
         iyz="0"
-        izz="0.0001" />
-    </inertial>
-    <visual>
-      <origin
-        xyz="0 0 0"
-        rpy="0 0 0" />
-      <geometry>
-        <mesh
-          filename="package://taurus_description/meshes/Rueda_izquierda_link.STL" />
+        izz="0.00001" />
+    </inertial>
+    <visual>
+      <origin
+        xyz="0 0 0"
+        rpy="0 0 0" />
+      <geometry>
+        <mesh
+          filename="package://taurus_description/meshes/rueda_izquierda_link.STL" />
       </geometry>
       <material
@@ -155,11 +152,10 @@
         rpy="0 0 0" />
       <geometry>
-        <mesh
-          filename="package://taurus_description/meshes/Rueda_izquierda_link.STL" />
-      </geometry>
-    </collision>
-  </link>
-  <joint
-    name="Rueda_izquierda_joint"
+        <cylinder radius="0.015" length="0.016"/>
+      </geometry>
+    </collision>
+  </link>
+  <joint
+    name="rueda_izquierda_joint"
     type="continuous">
     <origin
@@ -169,17 +165,16 @@
       link="base_link" />
     <child
-      link="Rueda_izquierda_link" />
+      link="rueda_izquierda_link" />
     <axis
       xyz="0 0 1" />
   </joint>
-   <gazebo reference="Rueda_izquierda_link">
+   <gazebo reference="rueda_izquierda_link">
     <mu1>200</mu1>
     <mu2>200</mu2>
     <kp>1000000</kp>
     <kd>1</kd>
-    <material>Gazebo/Gray</material>
-  </gazebo>
-  <link
-    name="Scan_link">
+  </gazebo>
+  <link
+    name="scan_link">
     <inertial>
       <origin
@@ -202,5 +197,5 @@
       <geometry>
         <mesh
-          filename="package://taurus_description/meshes/Scan_link.STL" />
+          filename="package://taurus_description/meshes/scan_link.STL" />
       </geometry>
       <material
@@ -216,10 +211,10 @@
       <geometry>
         <mesh
-          filename="package://taurus_description/meshes/Scan_link.STL" />
-      </geometry>
-    </collision>
-  </link>
-  <joint
-    name="Scan_joint"
+          filename="package://taurus_description/meshes/scan_link.STL" />
+      </geometry>
+    </collision>
+  </link>
+  <joint
+    name="scan_joint"
     type="fixed">
     <origin
@@ -229,10 +224,10 @@
       link="base_link" />
     <child
-      link="Scan_link" />
+      link="scan_link" />
     <axis
       xyz="0 0 0" />
   </joint>
   <link
-    name="Base_castor_link">
+    name="base_castor_link">
     <inertial>
       <origin
@@ -255,5 +250,5 @@
       <geometry>
         <mesh
-          filename="package://taurus_description/meshes/Base_castor_link.STL" />
+          filename="package://taurus_description/meshes/base_castor_link.STL" />
       </geometry>
       <material
@@ -269,10 +264,10 @@
       <geometry>
         <mesh
-          filename="package://taurus_description/meshes/Base_castor_link.STL" />
-      </geometry>
-    </collision>
-  </link>
-  <joint
-    name="Base_castor_joint"
+          filename="package://taurus_description/meshes/base_castor_link.STL" />
+      </geometry>
+    </collision>
+  </link>
+  <joint
+    name="base_castor_joint"
     type="fixed">
     <origin
@@ -282,10 +277,16 @@
       link="base_link" />
     <child
-      link="Base_castor_link" />
+      link="base_castor_link" />
     <axis
       xyz="0 0 0" />
   </joint>
-  <link
-    name="Caster_ball_link">
+    <gazebo reference="base_castor_link">
+    <mu1>0.1</mu1>
+    <mu2>0.1</mu2>
+    <kp>1000000</kp>
+    <kd>1</kd>
+  </gazebo>
+  <link
+    name="caster_ball_link">
     <inertial>
       <origin
@@ -293,20 +294,20 @@
         rpy="0 0 0" />
       <mass
-        value="0.002" />
-      <inertia
-        ixx="0.0004"
+        value="0.06" />
+      <inertia
+        ixx="0.00004"
         ixy="0"
         ixz="0"
-        iyy="0.0004"
+        iyy="0.00004"
         iyz="0"
-        izz="0.00001" />
-    </inertial>
-    <visual>
-      <origin
-        xyz="0 0 0"
-        rpy="0 0 0" />
-      <geometry>
-        <mesh
-          filename="package://taurus_description/meshes/Caster_ball_link.STL" />
+        izz="0.000001" />
+    </inertial>
+    <visual>
+      <origin
+        xyz="0 0 0"
+        rpy="0 0 0" />
+      <geometry>
+        <mesh
+          filename="package://taurus_description/meshes/caster_ball_link.STL" />
       </geometry>
       <material
@@ -321,30 +322,20 @@
         rpy="0 0 0" />
       <geometry>
-        <mesh
-          filename="package://taurus_description/meshes/Caster_ball_link.STL" />
-      </geometry>
-    </collision>
-  </link>
-    <gazebo reference="Caster_ball_link">
-    <mu1>100000</mu1>
-    <mu2>100000</mu2>
-    <kd>10.0</kd>
-    <minDepth>0.001</minDepth>
-    <maxVel>0.1</maxVel>
-    <fdir1>0 1 0</fdir1>
-    <fdir2>1 0 0</fdir2>
-  </gazebo>
-  <joint
-    name="Caster_ball_joint"
-    type="revolute">
+        <sphere radius="0.005"/>
+      </geometry>
+    </collision>
+  </link>
+  <joint
+    name="caster_ball_joint"
+    type="fixed">
     <origin
       xyz="-1.325E-05 -3.8318E-05 -0.004121"
       rpy="-1.5708 0 0" />
     <parent
-      link="Base_castor_link" />
-    <child
-      link="Caster_ball_link" />
+      link="base_castor_link" />
+    <child
+      link="caster_ball_link" />
     <axis
-      xyz="0 0 1" />
+      xyz="0 0 0" />
     <limit
       lower="0"
@@ -353,4 +344,10 @@
       velocity="0" />
   </joint>
+  <gazebo reference="caster_ball_link">
+    <mu1>0.1</mu1>
+    <mu2>0.1</mu2>
+    <kp>1000000</kp>
+    <kd>1</kd>
+  </gazebo>
   <link name="imu_link"/>
   <joint
@@ -364,9 +361,7 @@
     <child
       link="imu_link" />
-    <axis
-      xyz="1 0 0" />
   </joint>
   <!--LIDAR CONFIGURATION-->
-  <gazebo reference="Scan_link">
+  <gazebo reference="scan_link">
     <sensor name="lidar" type="ray">
       <always_on>true</always_on>
@@ -398,9 +393,9 @@
         </ros>
         <output_type>sensor_msgs/LaserScan</output_type>
-        <frame_name>Scan_link</frame_name>
+        <frame_name>scan_link</frame_name>
       </plugin>
     </sensor>
   </gazebo>
-  <gazebo reference="Scan_link">
+  <gazebo reference="scan_link">
     <mu1>0.1</mu1>
     <mu2>0.1</mu2>
@@ -434,9 +429,9 @@
       <update_rate>100</update_rate>
       <!-- wheels -->
-      <left_joint>Rueda_izquierda_joint</left_joint>
-      <right_joint>Rueda_derecha_joint</right_joint>
+      <left_joint>rueda_izquierda_joint</left_joint>
+      <right_joint>rueda_derecha_joint</right_joint>
       <!-- kinematics -->
       <wheel_separation>0.07</wheel_separation>
-      <wheel_diameter>0.016</wheel_diameter>
+      <wheel_diameter>0.030</wheel_diameter>
       <!-- limits -->
       <max_wheel_torque>20</max_wheel_torque>
@@ -462,3 +457,11 @@
     </plugin>
   </gazebo>
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